File: electronics_24wp/tca.sch (KiCad schematic (older format))
At the start: 26 parts, among them IC1 ATMEGA328-A, P1 CONN_2, P2 CONN_3X2, U1 SD_CARD, U2 LD1117S33, Y1 RESONATEUR

Commit message: Renamed electronic CAD folder.
Parts:
- C1, C2, C3, C4, C5: symbol C -> C-RESCUE-tca
- ERR1, FIN1, ON1: symbol LED -> LED-RESCUE-tca
- IC1: symbol ATMEGA328-A -> ATMEGA328-A-RESCUE-tca
- R1, R15, R16, R17, R18, R19, R2, R_ERR1, R_FIN1, R_ON1: symbol R -> R-RESCUE-tca
Changed lines of the file:
@@
 EESchema Schematic File Version 2
+LIBS:tca-rescue
 LIBS:power
 LIBS:device
@@
 LIBS:memory
 LIBS:xilinx
-LIBS:special
 LIBS:microcontrollers
 LIBS:dsp
@@
 LIBS:myParts
 LIBS:tca-cache
-EELAYER 27 0
+EELAYER 25 0
 EELAYER END
 $Descr USLetter 11000 8500
@@
 SS
 $Comp
-L GND #PWR01
+L GND-RESCUE-tca #PWR01
 U 1 1 5358B074
 P 2450 2800
@@
 $EndComp
 $Comp
-L C C5
+L C-RESCUE-tca C5
 U 1 1 535704C8
 P 3300 6600
@@
 $EndComp
 $Comp
-L C C3
+L C-RESCUE-tca C3
 U 1 1 535704B9
 P 1550 6600
@@
 ERR
 $Comp
-L R R_FIN1
+L R-RESCUE-tca R_FIN1
 U 1 1 5356ED9C
 P 4150 6850
@@
 $EndComp
 $Comp
-L R R_ERR1
+L R-RESCUE-tca R_ERR1
 U 1 1 5356ED8D
 P 4150 6550
@@
 $EndComp
 $Comp
-L R R_ON1
+L R-RESCUE-tca R_ON1
 U 1 1 5356ED7E
 P 4150 6250
@@
 ERR
 $Comp
-L LED FIN1
+L LED-RESCUE-tca FIN1
 U 1 1 5356E78D
 P 4750 6850
@@
 $EndComp
 $Comp
-L LED ERR1
+L LED-RESCUE-tca ERR1
 U 1 1 5356E77E
 P 4750 6550
@@
 $EndComp
 $Comp
-L LED ON1
+L LED-RESCUE-tca ON1
 U 1 1 5356E76F
 P 4750 6250
@@
 $EndComp
 $Comp
-L GND #PWR02
+L GND-RESCUE-tca #PWR02
 U 1 1 5356E577
 P 5100 7300
@@
 VCC
 $Comp
-L GND #PWR03
+L GND-RESCUE-tca #PWR03
 U 1 1 52166F83
 P 4300 4400
@@
 NoConn ~ 1350 4000
 $Comp
-L C C2
+L C-RESCUE-tca C2
 U 1 1 52150FEA
 P 1050 3700
@@
 $EndComp
 $Comp
-L C C1
+L C-RESCUE-tca C1
 U 1 1 52150FDD
 P 1050 3500
@@
 $EndComp
 $Comp
-L GND #PWR04
+L GND-RESCUE-tca #PWR04
 U 1 1 52150FBD
 P 800 5850
@@
 $EndComp
 $Comp
-L ATMEGA328-A IC1
+L ATMEGA328-A-RESCUE-tca IC1
 U 1 1 52150E25
 P 2250 4500
@@
 MOSI
 $Comp
-L R R1
+L R-RESCUE-tca R1
 U 1 1 5214E00C
 P 4500 7600
@@
 VCC
 $Comp
-L GND #PWR05
+L GND-RESCUE-tca #PWR05
 U 1 1 5214D884
 P 5050 5650
@@
 MISO
 $Comp
-L GND #PWR06
+L GND-RESCUE-tca #PWR06
 U 1 1 5214D369
 P 1250 6850
@@
 $EndSheet
 $Comp
-L R R2
+L R-RESCUE-tca R2
 U 1 1 5363149A
 P 6150 2900
@@
 $EndComp
 $Comp
-L C C4
+L C-RESCUE-tca C4
 U 1 1 53AA0322
 P 2250 6600
@@
 	2450 2150 2350 2150
 $Comp
-L R R15
+L R-RESCUE-tca R15
 U 1 1 53AA1B37
 P 2750 1400
@@
 $EndComp
 $Comp
-L R R16
+L R-RESCUE-tca R16
 U 1 1 53AA1B5A
 P 2950 1400
@@
 $EndComp
 $Comp
-L R R17
+L R-RESCUE-tca R17
 U 1 1 53AA1B60
 P 3150 1400
@@
 $EndComp
 $Comp
-L R R18
+L R-RESCUE-tca R18
 U 1 1 53AA1B66
 P 3350 1400
@@
 $EndComp
 $Comp
-L R R19
+L R-RESCUE-tca R19
 U 1 1 53AA1B6C
 P 3550 1400
