File: electronics_24wp/tlcs_1-3.sch (KiCad schematic (older format))
At the start: 57 parts, among them U3 TLC5941, U4 TLC5941, U5 TLC5941

Commit message: Renamed electronic CAD folder.
Parts:
- C6, C7, C8: symbol C -> C-RESCUE-tca
- D1, D10, D11, D12, D13, D14, D15, D16, D17, D18, D19, D2, D20, D21, D22, D23, D24, D25, D26, D27, D28, D29, D3, D30, D31, D32, D33, D34, D35, D36, D37, D38, D39, D4, D40, D41, D42, D43, D44, D45, D46, D47, D48, D5, D6, D7, D8, D9: symbol LED -> LED-RESCUE-tca
- R3, R4, R5: symbol R -> R-RESCUE-tca
Changed lines of the file:
@@
 EESchema Schematic File Version 2
+LIBS:tca-rescue
 LIBS:power
 LIBS:device
@@
 LIBS:memory
 LIBS:xilinx
-LIBS:special
 LIBS:microcontrollers
 LIBS:dsp
@@
 LIBS:myParts
 LIBS:tca-cache
-EELAYER 27 0
+EELAYER 25 0
 EELAYER END
 $Descr A4 11693 8268
@@
 NoConn ~ 3750 6100
 $Comp
-L GND #PWR07
+L GND-RESCUE-tca #PWR07
 U 1 1 53AA0802
 P 4600 5350
@@
 $EndComp
 $Comp
-L GND #PWR08
+L GND-RESCUE-tca #PWR08
 U 1 1 53AA0803
 P 1850 5550
@@
 $EndComp
 $Comp
-L R R5
+L R-RESCUE-tca R5
 U 1 1 5363017A
 P 4200 5700
@@
 $EndComp
 $Comp
-L C C8
+L C-RESCUE-tca C8
 U 1 1 53630180
 P 4050 5400
@@
 NoConn ~ 3750 3750
 $Comp
-L GND #PWR09
+L GND-RESCUE-tca #PWR09
 U 1 1 53AA0804
 P 4600 3000
@@
 $EndComp
 $Comp
-L GND #PWR010
+L GND-RESCUE-tca #PWR010
 U 1 1 5363096C
 P 1850 3200
@@
 $EndComp
 $Comp
-L R R4
+L R-RESCUE-tca R4
 U 1 1 5363096D
 P 4200 3350
@@
 $EndComp
 $Comp
-L C C7
+L C-RESCUE-tca C7
 U 1 1 53AA0807
 P 4050 3050
@@
 NoConn ~ 3750 1500
 $Comp
-L GND #PWR011
+L GND-RESCUE-tca #PWR011
 U 1 1 53AA0808
 P 4600 750
@@
 $EndComp
 $Comp
-L GND #PWR012
+L GND-RESCUE-tca #PWR012
 U 1 1 53630970
 P 1850 950
@@
 $EndComp
 $Comp
-L R R3
+L R-RESCUE-tca R3
 U 1 1 53630971
 P 4200 1100
@@
 $EndComp
 $Comp
-L C C6
+L C-RESCUE-tca C6
 U 1 1 53630972
 P 4050 800
@@
 	4550 6100 4550 6900
 $Comp
-L LED D1
+L LED-RESCUE-tca D1
 U 1 1 53AB4729
 P 1600 1600
@@
 $EndComp
 $Comp
-L LED D2
+L LED-RESCUE-tca D2
 U 1 1 53AB4736
 P 1600 1700
@@
 $EndComp
 $Comp
-L LED D3
+L LED-RESCUE-tca D3
 U 1 1 53AB473C
 P 1600 1800
@@
 $EndComp
 $Comp
-L LED D4
+L LED-RESCUE-tca D4
 U 1 1 53AB4742
 P 1600 1900
@@
 $EndComp
 $Comp
-L LED D5
+L LED-RESCUE-tca D5
 U 1 1 53AB4748
 P 1600 2000
@@
 $EndComp
 $Comp
-L LED D6
+L LED-RESCUE-tca D6
 U 1 1 53AB474E
 P 1600 2100
@@
 $EndComp
 $Comp
-L LED D7
+L LED-RESCUE-tca D7
 U 1 1 53AB4754
 P 1600 2200
@@
 $EndComp
 $Comp
-L LED D8
+L LED-RESCUE-tca D8
 U 1 1 53AB475A
 P 1600 2300
@@
 $EndComp
 $Comp
-L LED D9
+L LED-RESCUE-tca D9
 U 1 1 53AB4760
 P 1600 3850
@@
 $EndComp
 $Comp
-L LED D10
+L LED-RESCUE-tca D10
 U 1 1 53AB4766
 P 1600 3950
@@
 $EndComp
 $Comp
-L LED D11
+L LED-RESCUE-tca D11
 U 1 1 53AB476C
 P 1600 4050
@@
 $EndComp
 $Comp
-L LED D12
+L LED-RESCUE-tca D12
 U 1 1 53AB4772
 P 1600 4150
@@
 $EndComp
 $Comp
-L LED D13
+L LED-RESCUE-tca D13
 U 1 1 53AB4778
 P 1600 4250
@@
 $EndComp
 $Comp
-L LED D14
+L LED-RESCUE-tca D14
 U 1 1 53AB477E
 P 1600 4350
@@
 $EndComp
 $Comp
-L LED D15
+L LED-RESCUE-tca D15
 U 1 1 53AB4784
 P 1600 4450
@@
 $EndComp
 $Comp
-L LED D16
+L LED-RESCUE-tca D16
 U 1 1 53AB478A
 P 1600 4550
@@
 $EndComp
 $Comp
-L LED D17
+L LED-RESCUE-tca D17
 U 1 1 53AB47B8
 P 1600 6200
@@
 $EndComp
 $Comp
-L LED D18
+L LED-RESCUE-tca D18
 U 1 1 53AB47BE
 P 1600 6300
@@
 $EndComp
 $Comp
-L LED D19
+L LED-RESCUE-tca D19
 U 1 1 53AB47C4
 P 1600 6400
@@
 $EndComp
 $Comp
-L LED D20
+L LED-RESCUE-tca D20
 U 1 1 53AB47CA
 P 1600 6500
@@
 $EndComp
 $Comp
-L LED D21
+L LED-RESCUE-tca D21
 U 1 1 53AB47D0
 P 1600 6600
@@
 $EndComp
 $Comp
-L LED D22
+L LED-RESCUE-tca D22
 U 1 1 53AB47D6
 P 1600 6700
@@
 $EndComp
 $Comp
-L LED D23
+L LED-RESCUE-tca D23
 U 1 1 53AB47DC
 P 1600 6800
@@
 $EndComp
 $Comp
-L LED D24
+L LED-RESCUE-tca D24
 U 1 1 53AB47E2
 P 1600 6900
@@
 $EndComp
 $Comp
-L LED D25
+L LED-RESCUE-tca D25
 U 1 1 53AB47E8
 P 4250 1600
@@
 $EndComp
 $Comp
-L LED D26
+L LED-RESCUE-tca D26
 U 1 1 53AB47EE
 P 4250 1700
@@
 $EndComp
 $Comp
-L LED D27
+L LED-RESCUE-tca D27
 U 1 1 53AB47F4
 P 4250 1800
@@
 $EndComp
 $Comp
-L LED D28
+L LED-RESCUE-tca D28
 U 1 1 53AB47FA
 P 4250 1900
@@
 $EndComp
 $Comp
-L LED D29
+L LED-RESCUE-tca D29
 U 1 1 53AB4800
 P 4250 2000
@@
 $EndComp
 $Comp
-L LED D30
+L LED-RESCUE-tca D30
 U 1 1 53AB4806
 P 4250 2100
@@
 $EndComp
 $Comp
-L LED D31
+L LED-RESCUE-tca D31
 U 1 1 53AB480C
 P 4250 2200
@@
 $EndComp
 $Comp
-L LED D32
+L LED-RESCUE-tca D32
 U 1 1 53AB4812
 P 4250 2300
@@
 $EndComp
 $Comp
-L LED D33
+L LED-RESCUE-tca D33
 U 1 1 53AB4820
 P 4250 3850
@@
 $EndComp
 $Comp
-L LED D34
+L LED-RESCUE-tca D34
 U 1 1 53AB4826
 P 4250 3950
@@
 $EndComp
 $Comp
-L LED D35
+L LED-RESCUE-tca D35
 U 1 1 53AB482C
 P 4250 4050
@@
 $EndComp
 $Comp
-L LED D36
+L LED-RESCUE-tca D36
 U 1 1 53AB4832
 P 4250 4150
@@
 $EndComp
 $Comp
-L LED D37
+L LED-RESCUE-tca D37
 U 1 1 53AB4838
 P 4250 4250
@@
 $EndComp
 $Comp
-L LED D38
+L LED-RESCUE-tca D38
 U 1 1 53AB483E
 P 4250 4350
@@
 $EndComp
 $Comp
-L LED D39
+L LED-RESCUE-tca D39
 U 1 1 53AB4844
 P 4250 4450
@@
 $EndComp
 $Comp
-L LED D40
+L LED-RESCUE-tca D40
 U 1 1 53AB484A
 P 4250 4550
@@
 $EndComp
 $Comp
-L LED D41
+L LED-RESCUE-tca D41
 U 1 1 53AB4850
 P 4250 6200
@@
 $EndComp
 $Comp
-L LED D42
+L LED-RESCUE-tca D42
 U 1 1 53AB4856
 P 4250 6300
@@
 $EndComp
 $Comp
-L LED D43
+L LED-RESCUE-tca D43
 U 1 1 53AB485C
 P 4250 6400
@@
 $EndComp
 $Comp
-L LED D44
+L LED-RESCUE-tca D44
 U 1 1 53AB4862
 P 4250 6500
@@
 $EndComp
 $Comp
-L LED D45
+L LED-RESCUE-tca D45
 U 1 1 53AB4868
 P 4250 6600
@@
 $EndComp
 $Comp
-L LED D46
+L LED-RESCUE-tca D46
 U 1 1 53AB486E
 P 4250 6700
@@
 $EndComp
 $Comp
-L LED D47
+L LED-RESCUE-tca D47
 U 1 1 53AB4874
 P 4250 6800
@@
 $EndComp
 $Comp
-L LED D48
+L LED-RESCUE-tca D48
 U 1 1 53AB487A
 P 4250 6900

Commit message: Changed names of kicad files.
Parts:
- C6, C7, C8: symbol C-RESCUE-tca -> C-RESCUE-lpa
- D1, D10, D11, D12, D13, D14, D15, D16, D17, D18, D19, D2, D20, D21, D22, D23, D24, D25, D26, D27, D28, D29, D3, D30, D31, D32, D33, D34, D35, D36, D37, D38, D39, D4, D40, D41, D42, D43, D44, D45, D46, D47, D48, D5, D6, D7, D8, D9: symbol LED-RESCUE-tca -> LED-RESCUE-lpa
- R3, R4, R5: symbol R-RESCUE-tca -> R-RESCUE-lpa
Changed lines of the file:
@@
 EESchema Schematic File Version 2
-LIBS:tca-rescue
+LIBS:lpa-rescue
 LIBS:power
 LIBS:device
@@
 LIBS:valves
 LIBS:myParts
-LIBS:tca-cache
+LIBS:lpa-cache
 EELAYER 25 0
 EELAYER END
@@
 NoConn ~ 3750 6100
 $Comp
-L GND-RESCUE-tca #PWR07
+L GND-RESCUE-lpa #PWR07
 U 1 1 53AA0802
 P 4600 5350
@@
 $EndComp
 $Comp
-L GND-RESCUE-tca #PWR08
+L GND-RESCUE-lpa #PWR08
 U 1 1 53AA0803
 P 1850 5550
@@
 $EndComp
 $Comp
-L R-RESCUE-tca R5
+L R-RESCUE-lpa R5
 U 1 1 5363017A
 P 4200 5700
@@
 $EndComp
 $Comp
-L C-RESCUE-tca C8
+L C-RESCUE-lpa C8
 U 1 1 53630180
 P 4050 5400
@@
 NoConn ~ 3750 3750
 $Comp
-L GND-RESCUE-tca #PWR09
+L GND-RESCUE-lpa #PWR09
 U 1 1 53AA0804
 P 4600 3000
@@
 $EndComp
 $Comp
-L GND-RESCUE-tca #PWR010
+L GND-RESCUE-lpa #PWR010
 U 1 1 5363096C
 P 1850 3200
@@
 $EndComp
 $Comp
-L R-RESCUE-tca R4
+L R-RESCUE-lpa R4
 U 1 1 5363096D
 P 4200 3350
@@
 $EndComp
 $Comp
-L C-RESCUE-tca C7
+L C-RESCUE-lpa C7
 U 1 1 53AA0807
 P 4050 3050
@@
 NoConn ~ 3750 1500
 $Comp
-L GND-RESCUE-tca #PWR011
+L GND-RESCUE-lpa #PWR011
 U 1 1 53AA0808
 P 4600 750
@@
 $EndComp
 $Comp
-L GND-RESCUE-tca #PWR012
+L GND-RESCUE-lpa #PWR012
 U 1 1 53630970
 P 1850 950
@@
 $EndComp
 $Comp
-L R-RESCUE-tca R3
+L R-RESCUE-lpa R3
 U 1 1 53630971
 P 4200 1100
@@
 $EndComp
 $Comp
-L C-RESCUE-tca C6
+L C-RESCUE-lpa C6
 U 1 1 53630972
 P 4050 800
@@
 	4550 6100 4550 6900
 $Comp
-L LED-RESCUE-tca D1
+L LED-RESCUE-lpa D1
 U 1 1 53AB4729
 P 1600 1600
@@
 $EndComp
 $Comp
-L LED-RESCUE-tca D2
+L LED-RESCUE-lpa D2
 U 1 1 53AB4736
 P 1600 1700
@@
 $EndComp
 $Comp
-L LED-RESCUE-tca D3
+L LED-RESCUE-lpa D3
 U 1 1 53AB473C
 P 1600 1800
@@
 $EndComp
 $Comp
-L LED-RESCUE-tca D4
+L LED-RESCUE-lpa D4
 U 1 1 53AB4742
 P 1600 1900
@@
 $EndComp
 $Comp
-L LED-RESCUE-tca D5
+L LED-RESCUE-lpa D5
 U 1 1 53AB4748
 P 1600 2000
@@
 $EndComp
 $Comp
-L LED-RESCUE-tca D6
+L LED-RESCUE-lpa D6
 U 1 1 53AB474E
 P 1600 2100
@@
 $EndComp
 $Comp
-L LED-RESCUE-tca D7
+L LED-RESCUE-lpa D7
 U 1 1 53AB4754
 P 1600 2200
@@
 $EndComp
 $Comp
-L LED-RESCUE-tca D8
+L LED-RESCUE-lpa D8
 U 1 1 53AB475A
 P 1600 2300
@@
 $EndComp
 $Comp
-L LED-RESCUE-tca D9
+L LED-RESCUE-lpa D9
 U 1 1 53AB4760
 P 1600 3850
@@
 $EndComp
 $Comp
-L LED-RESCUE-tca D10
+L LED-RESCUE-lpa D10
 U 1 1 53AB4766
 P 1600 3950
@@
 $EndComp
 $Comp
-L LED-RESCUE-tca D11
+L LED-RESCUE-lpa D11
 U 1 1 53AB476C
 P 1600 4050
@@
 $EndComp
 $Comp
-L LED-RESCUE-tca D12
+L LED-RESCUE-lpa D12
 U 1 1 53AB4772
 P 1600 4150
@@
 $EndComp
 $Comp
-L LED-RESCUE-tca D13
+L LED-RESCUE-lpa D13
 U 1 1 53AB4778
 P 1600 4250
@@
 $EndComp
 $Comp
-L LED-RESCUE-tca D14
+L LED-RESCUE-lpa D14
 U 1 1 53AB477E
 P 1600 4350
@@
 $EndComp
 $Comp
-L LED-RESCUE-tca D15
+L LED-RESCUE-lpa D15
 U 1 1 53AB4784
 P 1600 4450
@@
 $EndComp
 $Comp
-L LED-RESCUE-tca D16
+L LED-RESCUE-lpa D16
 U 1 1 53AB478A
 P 1600 4550
@@
 $EndComp
 $Comp
-L LED-RESCUE-tca D17
+L LED-RESCUE-lpa D17
 U 1 1 53AB47B8
 P 1600 6200
@@
 $EndComp
 $Comp
-L LED-RESCUE-tca D18
+L LED-RESCUE-lpa D18
 U 1 1 53AB47BE
 P 1600 6300
@@
 $EndComp
 $Comp
-L LED-RESCUE-tca D19
+L LED-RESCUE-lpa D19
 U 1 1 53AB47C4
 P 1600 6400
@@
 $EndComp
 $Comp
-L LED-RESCUE-tca D20
+L LED-RESCUE-lpa D20
 U 1 1 53AB47CA
 P 1600 6500
@@
 $EndComp
 $Comp
-L LED-RESCUE-tca D21
+L LED-RESCUE-lpa D21
 U 1 1 53AB47D0
 P 1600 6600
@@
 $EndComp
 $Comp
-L LED-RESCUE-tca D22
+L LED-RESCUE-lpa D22
 U 1 1 53AB47D6
 P 1600 6700
@@
 $EndComp
 $Comp
-L LED-RESCUE-tca D23
+L LED-RESCUE-lpa D23
 U 1 1 53AB47DC
 P 1600 6800
@@
 $EndComp
 $Comp
-L LED-RESCUE-tca D24
+L LED-RESCUE-lpa D24
 U 1 1 53AB47E2
 P 1600 6900
@@
 $EndComp
 $Comp
-L LED-RESCUE-tca D25
+L LED-RESCUE-lpa D25
 U 1 1 53AB47E8
 P 4250 1600
@@
 $EndComp
 $Comp
-L LED-RESCUE-tca D26
+L LED-RESCUE-lpa D26
 U 1 1 53AB47EE
 P 4250 1700
@@
 $EndComp
 $Comp
-L LED-RESCUE-tca D27
+L LED-RESCUE-lpa D27
 U 1 1 53AB47F4
 P 4250 1800
@@
 $EndComp
 $Comp
-L LED-RESCUE-tca D28
+L LED-RESCUE-lpa D28
 U 1 1 53AB47FA
 P 4250 1900
@@
 $EndComp
 $Comp
-L LED-RESCUE-tca D29
+L LED-RESCUE-lpa D29
 U 1 1 53AB4800
 P 4250 2000
@@
 $EndComp
 $Comp
-L LED-RESCUE-tca D30
+L LED-RESCUE-lpa D30
 U 1 1 53AB4806
 P 4250 2100
@@
 $EndComp
 $Comp
-L LED-RESCUE-tca D31
+L LED-RESCUE-lpa D31
 U 1 1 53AB480C
 P 4250 2200
@@
 $EndComp
 $Comp
-L LED-RESCUE-tca D32
+L LED-RESCUE-lpa D32
 U 1 1 53AB4812
 P 4250 2300
@@
 $EndComp
 $Comp
-L LED-RESCUE-tca D33
+L LED-RESCUE-lpa D33
 U 1 1 53AB4820
 P 4250 3850
@@
 $EndComp
 $Comp
-L LED-RESCUE-tca D34
+L LED-RESCUE-lpa D34
 U 1 1 53AB4826
 P 4250 3950
@@
 $EndComp
 $Comp
-L LED-RESCUE-tca D35
+L LED-RESCUE-lpa D35
 U 1 1 53AB482C
 P 4250 4050
@@
 $EndComp
 $Comp
-L LED-RESCUE-tca D36
+L LED-RESCUE-lpa D36
 U 1 1 53AB4832
 P 4250 4150
@@
 $EndComp
 $Comp
-L LED-RESCUE-tca D37
+L LED-RESCUE-lpa D37
 U 1 1 53AB4838
 P 4250 4250
@@
 $EndComp
 $Comp
-L LED-RESCUE-tca D38
+L LED-RESCUE-lpa D38
 U 1 1 53AB483E
 P 4250 4350
@@
 $EndComp
 $Comp
-L LED-RESCUE-tca D39
+L LED-RESCUE-lpa D39
 U 1 1 53AB4844
 P 4250 4450
@@
 $EndComp
 $Comp
-L LED-RESCUE-tca D40
+L LED-RESCUE-lpa D40
 U 1 1 53AB484A
 P 4250 4550
@@
 $EndComp
 $Comp
-L LED-RESCUE-tca D41
+L LED-RESCUE-lpa D41
 U 1 1 53AB4850
 P 4250 6200
@@
 $EndComp
 $Comp
-L LED-RESCUE-tca D42
+L LED-RESCUE-lpa D42
 U 1 1 53AB4856
 P 4250 6300
@@
 $EndComp
 $Comp
-L LED-RESCUE-tca D43
+L LED-RESCUE-lpa D43
 U 1 1 53AB485C
 P 4250 6400
@@
 $EndComp
 $Comp
-L LED-RESCUE-tca D44
+L LED-RESCUE-lpa D44
 U 1 1 53AB4862
 P 4250 6500
@@
 $EndComp
 $Comp
-L LED-RESCUE-tca D45
+L LED-RESCUE-lpa D45
 U 1 1 53AB4868
 P 4250 6600
@@
 $EndComp
 $Comp
-L LED-RESCUE-tca D46
+L LED-RESCUE-lpa D46
 U 1 1 53AB486E
 P 4250 6700
@@
 $EndComp
 $Comp
-L LED-RESCUE-tca D47
+L LED-RESCUE-lpa D47
 U 1 1 53AB4874
 P 4250 6800
@@
 $EndComp
 $Comp
-L LED-RESCUE-tca D48
+L LED-RESCUE-lpa D48
 U 1 1 53AB487A
 P 4250 6900

Commit message: Improved footprint of TLCs.
Parts:
- U3, U4, U5: footprint TLC5940_THERMVIAS2 -> LPA_parts:TLC5940_THERMVIAS
Changed lines of the file:
@@
 F 0 "U5" H 3000 6150 50  0000 C CNN
 F 1 "TLC5941" H 3000 6350 50  0000 C CNN
-F 2 "TLC5940_THERMVIAS2" H 3000 6250 50  0001 C CNN
+F 2 "LPA_parts:TLC5940_THERMVIAS" H 3000 6250 50  0001 C CNN
 F 3 "DOCUMENTATION" H 3000 6250 50  0001 C CNN
 	1    3000 6250
@@
 F 0 "U4" H 3000 3800 50  0000 C CNN
 F 1 "TLC5941" H 3000 4000 50  0000 C CNN
-F 2 "TLC5940_THERMVIAS2" H 3000 3900 50  0001 C CNN
+F 2 "LPA_parts:TLC5940_THERMVIAS" H 3000 3900 50  0001 C CNN
 F 3 "DOCUMENTATION" H 3000 3900 50  0001 C CNN
 	1    3000 3900
@@
 F 0 "U3" H 3000 1550 50  0000 C CNN
 F 1 "TLC5941" H 3000 1750 50  0000 C CNN
-F 2 "TLC5940_THERMVIAS2" H 3000 1650 50  0001 C CNN
+F 2 "LPA_parts:TLC5940_THERMVIAS" H 3000 1650 50  0001 C CNN
 F 3 "DOCUMENTATION" H 3000 1650 50  0001 C CNN
 	1    3000 1650

Commit message: Streamlined library files for the electronic schematic.
Parts:
- C6, C7, C8: symbol C-RESCUE-lpa -> C
- D1, D10, D11, D12, D13, D14, D15, D16, D17, D18, D19, D2, D20, D21, D22, D23, D24, D25, D26, D27, D28, D29, D3, D30, D31, D32, D33, D34, D35, D36, D37, D38, D39, D4, D40, D41, D42, D43, D44, D45, D46, D47, D48, D5, D6, D7, D8, D9: symbol LED-RESCUE-lpa -> LED-INV
- R3, R4, R5: symbol R-RESCUE-lpa -> R
Changed lines of the file:
@@
 EESchema Schematic File Version 2
-LIBS:lpa-rescue
 LIBS:power
 LIBS:device
@@
 Connection ~ 4450 5200
 Wire Wire Line
-	3950 5700 3750 5700
+	3750 5700 4050 5700
 Wire Wire Line
 	3750 5600 4050 5600
@@
 Connection ~ 4450 2850
 Wire Wire Line
-	3950 3350 3750 3350
+	3750 3350 4050 3350
 Wire Wire Line
 	3750 3250 4050 3250
@@
 Connection ~ 4450 600
 Wire Wire Line
-	3950 1100 3750 1100
+	3750 1100 4050 1100
 Wire Wire Line
 	3750 1000 4050 1000
@@
 NoConn ~ 3750 6100
 $Comp
-L GND-RESCUE-lpa #PWR09
+L GND #PWR09
 U 1 1 53AA0802
 P 4600 5350
@@
 $EndComp
 $Comp
-L GND-RESCUE-lpa #PWR010
+L GND #PWR010
 U 1 1 53AA0803
 P 1850 5550
@@
 $EndComp
 $Comp
-L R-RESCUE-lpa R5
+L R R5
 U 1 1 5363017A
 P 4200 5700
@@
 $EndComp
 $Comp
-L C-RESCUE-lpa C8
+L C C8
 U 1 1 53630180
 P 4050 5400
@@
 NoConn ~ 3750 3750
 $Comp
-L GND-RESCUE-lpa #PWR011
+L GND #PWR011
 U 1 1 53AA0804
 P 4600 3000
@@
 $EndComp
 $Comp
-L GND-RESCUE-lpa #PWR012
+L GND #PWR012
 U 1 1 5363096C
 P 1850 3200
@@
 $EndComp
 $Comp
-L R-RESCUE-lpa R4
+L R R4
 U 1 1 5363096D
 P 4200 3350
@@
 $EndComp
 $Comp
-L C-RESCUE-lpa C7
+L C C7
 U 1 1 53AA0807
 P 4050 3050
@@
 NoConn ~ 3750 1500
 $Comp
-L GND-RESCUE-lpa #PWR013
+L GND #PWR013
 U 1 1 53AA0808
 P 4600 750
@@
 $EndComp
 $Comp
-L GND-RESCUE-lpa #PWR014
+L GND #PWR014
 U 1 1 53630970
 P 1850 950
@@
 $EndComp
 $Comp
-L R-RESCUE-lpa R3
+L R R3
 U 1 1 53630971
 P 4200 1100
@@
 $EndComp
 $Comp
-L C-RESCUE-lpa C6
+L C C6
 U 1 1 53630972
 P 4050 800
@@
 	4550 6100 4550 6900
 $Comp
-L LED-RESCUE-lpa D1
+L LED-INV D1
 U 1 1 53AB4729
 P 1600 1600
@@
 $EndComp
 $Comp
-L LED-RESCUE-lpa D2
+L LED-INV D2
 U 1 1 53AB4736
 P 1600 1700
@@
 $EndComp
 $Comp
-L LED-RESCUE-lpa D3
+L LED-INV D3
 U 1 1 53AB473C
 P 1600 1800
@@
 $EndComp
 $Comp
-L LED-RESCUE-lpa D4
+L LED-INV D4
 U 1 1 53AB4742
 P 1600 1900
@@
 $EndComp
 $Comp
-L LED-RESCUE-lpa D5
+L LED-INV D5
 U 1 1 53AB4748
 P 1600 2000
@@
 $EndComp
 $Comp
-L LED-RESCUE-lpa D6
+L LED-INV D6
 U 1 1 53AB474E
 P 1600 2100
@@
 $EndComp
 $Comp
-L LED-RESCUE-lpa D7
+L LED-INV D7
 U 1 1 53AB4754
 P 1600 2200
@@
 $EndComp
 $Comp
-L LED-RESCUE-lpa D8
+L LED-INV D8
 U 1 1 53AB475A
 P 1600 2300
@@
 $EndComp
 $Comp
-L LED-RESCUE-lpa D9
+L LED-INV D9
 U 1 1 53AB4760
 P 1600 3850
@@
 $EndComp
 $Comp
-L LED-RESCUE-lpa D10
+L LED-INV D10
 U 1 1 53AB4766
 P 1600 3950
@@
 $EndComp
 $Comp
-L LED-RESCUE-lpa D11
+L LED-INV D11
 U 1 1 53AB476C
 P 1600 4050
@@
 $EndComp
 $Comp
-L LED-RESCUE-lpa D12
+L LED-INV D12
 U 1 1 53AB4772
 P 1600 4150
@@
 $EndComp
 $Comp
-L LED-RESCUE-lpa D13
+L LED-INV D13
 U 1 1 53AB4778
 P 1600 4250
@@
 $EndComp
 $Comp
-L LED-RESCUE-lpa D14
+L LED-INV D14
 U 1 1 53AB477E
 P 1600 4350
@@
 $EndComp
 $Comp
-L LED-RESCUE-lpa D15
+L LED-INV D15
 U 1 1 53AB4784
 P 1600 4450
@@
 $EndComp
 $Comp
-L LED-RESCUE-lpa D16
+L LED-INV D16
 U 1 1 53AB478A
 P 1600 4550
@@
 $EndComp
 $Comp
-L LED-RESCUE-lpa D17
+L LED-INV D17
 U 1 1 53AB47B8
 P 1600 6200
@@
 $EndComp
 $Comp
-L LED-RESCUE-lpa D18
+L LED-INV D18
 U 1 1 53AB47BE
 P 1600 6300
@@
 $EndComp
 $Comp
-L LED-RESCUE-lpa D19
+L LED-INV D19
 U 1 1 53AB47C4
 P 1600 6400
@@
 $EndComp
 $Comp
-L LED-RESCUE-lpa D20
+L LED-INV D20
 U 1 1 53AB47CA
 P 1600 6500
@@
 $EndComp
 $Comp
-L LED-RESCUE-lpa D21
+L LED-INV D21
 U 1 1 53AB47D0
 P 1600 6600
@@
 $EndComp
 $Comp
-L LED-RESCUE-lpa D22
+L LED-INV D22
 U 1 1 53AB47D6
 P 1600 6700
@@
 $EndComp
 $Comp
-L LED-RESCUE-lpa D23
+L LED-INV D23
 U 1 1 53AB47DC
 P 1600 6800
@@
 $EndComp
 $Comp
-L LED-RESCUE-lpa D24
+L LED-INV D24
 U 1 1 53AB47E2
 P 1600 6900
@@
 $EndComp
 $Comp
-L LED-RESCUE-lpa D25
+L LED-INV D25
 U 1 1 53AB47E8
 P 4250 1600
@@
 $EndComp
 $Comp
-L LED-RESCUE-lpa D26
+L LED-INV D26
 U 1 1 53AB47EE
 P 4250 1700
@@
 $EndComp
 $Comp
-L LED-RESCUE-lpa D27
+L LED-INV D27
 U 1 1 53AB47F4
 P 4250 1800
@@
 $EndComp
 $Comp
-L LED-RESCUE-lpa D28
+L LED-INV D28
 U 1 1 53AB47FA
 P 4250 1900
@@
 $EndComp
 $Comp
-L LED-RESCUE-lpa D29
+L LED-INV D29
 U 1 1 53AB4800
 P 4250 2000
@@
 $EndComp
 $Comp
-L LED-RESCUE-lpa D30
+L LED-INV D30
 U 1 1 53AB4806
 P 4250 2100
@@
 $EndComp
 $Comp
-L LED-RESCUE-lpa D31
+L LED-INV D31
 U 1 1 53AB480C
 P 4250 2200
@@
 $EndComp
 $Comp
-L LED-RESCUE-lpa D32
+L LED-INV D32
 U 1 1 53AB4812
 P 4250 2300
@@
 $EndComp
 $Comp
-L LED-RESCUE-lpa D33
+L LED-INV D33
 U 1 1 53AB4820
 P 4250 3850
@@
 $EndComp
 $Comp
-L LED-RESCUE-lpa D34
+L LED-INV D34
 U 1 1 53AB4826
 P 4250 3950
@@
 $EndComp
 $Comp
-L LED-RESCUE-lpa D35
+L LED-INV D35
 U 1 1 53AB482C
 P 4250 4050
@@
 $EndComp
 $Comp
-L LED-RESCUE-lpa D36
+L LED-INV D36
 U 1 1 53AB4832
 P 4250 4150
@@
 $EndComp
 $Comp
-L LED-RESCUE-lpa D37
+L LED-INV D37
 U 1 1 53AB4838
 P 4250 4250
@@
 $EndComp
 $Comp
-L LED-RESCUE-lpa D38
+L LED-INV D38
 U 1 1 53AB483E
 P 4250 4350
@@
 $EndComp
 $Comp
-L LED-RESCUE-lpa D39
+L LED-INV D39
 U 1 1 53AB4844
 P 4250 4450
@@
 $EndComp
 $Comp
-L LED-RESCUE-lpa D40
+L LED-INV D40
 U 1 1 53AB484A
 P 4250 4550
@@
 $EndComp
 $Comp
-L LED-RESCUE-lpa D41
+L LED-INV D41
 U 1 1 53AB4850
 P 4250 6200
@@
 $EndComp
 $Comp
-L LED-RESCUE-lpa D42
+L LED-INV D42
 U 1 1 53AB4856
 P 4250 6300
@@
 $EndComp
 $Comp
-L LED-RESCUE-lpa D43
+L LED-INV D43
 U 1 1 53AB485C
 P 4250 6400
@@
 $EndComp
 $Comp
-L LED-RESCUE-lpa D44
+L LED-INV D44
 U 1 1 53AB4862
 P 4250 6500
@@
 $EndComp
 $Comp
-L LED-RESCUE-lpa D45
+L LED-INV D45
 U 1 1 53AB4868
 P 4250 6600
@@
 $EndComp
 $Comp
-L LED-RESCUE-lpa D46
+L LED-INV D46
 U 1 1 53AB486E
 P 4250 6700
@@
 $EndComp
 $Comp
-L LED-RESCUE-lpa D47
+L LED-INV D47
 U 1 1 53AB4874
 P 4250 6800
@@
 $EndComp
 $Comp
-L LED-RESCUE-lpa D48
+L LED-INV D48
 U 1 1 53AB487A
 P 4250 6900
@@
 	-1   0    0    -1
 $EndComp
+Wire Wire Line
+	4050 650  4050 600
+Wire Wire Line
+	4050 1000 4050 950
+Wire Wire Line
+	4050 2850 4050 2900
+Wire Wire Line
+	4050 3250 4050 3200
+Wire Wire Line
+	4050 5200 4050 5250
+Wire Wire Line
+	4050 5600 4050 5550
+Wire Wire Line
+	4450 5700 4350 5700
+Wire Wire Line
+	4350 3350 4450 3350
+Wire Wire Line
+	4350 1100 4450 1100
 $EndSCHEMATC

Commit message: Assigned footprint to LED sockets.
Parts:
- D1, D10, D11, D12, D13, D14, D15, D16, D17, D18, D19, D2, D20, D21, D22, D23, D24, D25, D26, D27, D28, D29, D3, D30, D31, D32, D33, D34, D35, D36, D37, D38, D39, D4, D40, D41, D42, D43, D44, D45, D46, D47, D48, D5, D6, D7, D8, D9: footprint ~ -> LPA_parts:PCV220_LEDSOCKET

Commit message: Streamlined layout libraries.
Parts:
- C6, C7, C8, R3, R4, R5: footprint SM0805 -> LPA_parts:SM0805
- D1, D10, D11, D12, D13, D14, D15, D16, D17, D18, D19, D2, D20, D21, D22, D23, D24, D25, D26, D27, D28, D29, D3, D30, D31, D32, D33, D34, D35, D36, D37, D38, D39, D4, D40, D41, D42, D43, D44, D45, D46, D47, D48, D5, D6, D7, D8, D9: footprint LPA_parts:PCV220_LEDSOCKET -> LPA_parts:PCV220_LED_SOCKET
- U3, U4, U5: footprint LPA_parts:TLC5940_THERMVIAS -> LPA_parts:TLC5941
